File: UltrasonicPCB.kicad_pcb (KiCad board)
At the start: 2 copper layers, 65 x 64.2 mm, 11 parts, among them J2 Conn_01x07

Commit message: Fixed Ultrasonic Sides
Parts:
- U1, U5: moved to B.Cu
- moved D1 37.5 mm to (101.4, 97.9), turned to -90 degrees
- moved U5 10.2 mm to (146.2, 93.6)
- moved U3 10.1 mm to (131.3, 70.1), turned to -90 degrees
- turned U1 to 0 degrees
Routing:
- net Net-(D1-A): track 59.9 -> 5.13 mm
- net GND: track 167.8 -> 129.8 mm
- net Net-(J2-Pin_6): track 17.6 -> 54.9 mm, vias 1 -> 0
- net ECHO: track 161.9 -> 126.7 mm
- net 5V: track 148.3 -> 118.3 mm
- net TRIG2: track 30.6 -> 46.9 mm
- net Net-(D3-A): track 38.6 -> 54.1 mm
- net Net-(D2-A): track 44.6 -> 30.9 mm
- net Net-(D4-A): track 19.6 -> 6.66 mm
- net TRIG3: track 35.8 -> 43.6 mm
- net TRIG4: track 49.6 -> 44.3 mm
