File: UltrasonicPCB.kicad_pcb (KiCad board)
At the start: 2 copper layers, 65 x 64.2 mm, 11 parts, among them J2 Conn_01x07

Commit message: Remake the PCB
Parts:
- added H1: MountingHole, MountingHole:MountingHole_3.2mm_M3_DIN965_Pad, F.Cu at (-11.5, 55.0)
- added H2: MountingHole, MountingHole:MountingHole_3.2mm_M3_DIN965_Pad, F.Cu at (-11.5, 6.00)
- added H3: MountingHole, MountingHole:MountingHole_3.2mm_M3_DIN965_Pad, F.Cu at (5.50, 58.5)
- added H4: MountingHole, MountingHole:MountingHole_3.2mm_M3_DIN965_Pad, F.Cu at (5.50, 2.50)
- added H5: MountingHole, MountingHole:MountingHole_3.2mm_M3_DIN965_Pad, F.Cu at (29.5, 58.5)
- added H6: MountingHole, MountingHole:MountingHole_3.2mm_M3_DIN965_Pad, F.Cu at (29.5, 2.50)
- added H7: MountingHole, MountingHole:MountingHole_3.2mm_M3_DIN965_Pad, F.Cu at (46.5, 55.0)
- added H8: MountingHole, MountingHole:MountingHole_3.2mm_M3_DIN965_Pad, F.Cu at (46.5, 6.00)
- J2, U1, U5: moved to F.Cu
- R1: value R -> 10k
- R2: value R -> 15k
- U2, U3: moved to B.Cu
- moved D4 153.3 mm to (15.5, 29.5), turned to 0 degrees
- moved D3 145.3 mm to (15.5, 27.0), turned to 0 degrees
- moved D2 140.2 mm to (15.5, 34.5), turned to 0 degrees
- moved U1 134.0 mm to (-2.50, 25.4)
- moved J2 132.5 mm to (-11.0, 64.5), turned to 90 degrees
- moved U3 128.3 mm to (22.6, 1.86), turned to 90 degrees
- moved R1 124.2 mm to (-2.02, 49.4)
- moved R2 124.2 mm to (-2.00, 47.0)
- moved U5 123.3 mm to (37.5, 35.6)
- moved U2 119.9 mm to (22.6, 59.1)
- moved D1 108.3 mm to (15.5, 32.0), turned to 180 degrees
Routing:
- net GND: track 129.8 -> 0.00 mm
- net ECHO: track 126.7 -> 31.4 mm
- net 5V: track 118.3 -> 162.0 mm
- net Net-(J2-Pin_6): track 54.9 -> 18.4 mm
- net TRIG3: track 43.6 -> 73.3 mm
- net Net-(D3-A): track 54.1 -> 25.3 mm, vias 0 -> 1
- net TRIG1: track 14.0 -> 41.0 mm
- net Net-(D4-A): track 6.66 -> 20.8 mm
- net TRIG4: track 44.3 -> 57.6 mm, vias 0 -> 1
- net TRIG2: track 46.9 -> 34.4 mm
- net Net-(D1-A): track 5.13 -> 16.9 mm
Other:
- board size 65 x 64.2 mm -> 65 x 69.1 mm

Commit message: continuation
Parts:
- U3: moved to F.Cu
- moved U2 142.9 mm to (149.6, 124.7)
- moved U1 141.8 mm to (126.5, 84.2)
- moved D2 140.0 mm to (142.5, 93.3)
- moved D3 140.0 mm to (142.5, 85.8)
- moved D4 140.0 mm to (142.5, 88.3)
- moved H1 140.0 mm to (115.5, 113.8)
- moved H2 140.0 mm to (115.5, 64.8)
- moved H3 140.0 mm to (132.5, 117.3)
- moved H4 140.0 mm to (132.5, 61.3)
- moved H5 140.0 mm to (156.5, 117.3)
- moved H6 140.0 mm to (156.5, 61.3)
- moved H7 140.0 mm to (173.5, 113.8)
- moved H8 140.0 mm to (173.5, 64.8)
- moved J2 140.0 mm to (116.0, 123.3)
- moved R1 140.0 mm to (125.0, 108.2)
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Routing:
- net 5V: track 162.0 -> 140.8 mm
- net TRIG3: track 73.3 -> 66.6 mm
- net TRIG2: track 34.4 -> 31.0 mm
- net Net-(D3-A): track 25.3 -> 22.0 mm, vias 1 -> 0
- net Net-(D4-A): track 20.8 -> 18.8 mm
- net Net-(D1-A): track 16.9 -> 14.9 mm, vias 0 -> 1
- net TRIG1: track 41.0 -> 39.9 mm
Other:
- outline, holes or cut-outs redrawn
